File: PCB/mainboard/mainboard.sch (EAGLE design)
At the start: 18 parts

Commit message: Fix fonts and switch.
This commit will fix two issue.
First, use the vector font because the true type is different from prited.
Second, replace the slide switch because we used the wrong one.
Parts:
- S1: device switch:255SB -> switch:M251
Changed lines of the file:
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@@
 <part name="MBED" library="MBED_v2.1" deviceset="MBED_NXP_LPC1768" device=""/>
 <part name="ZX2" library="con-3m" deviceset="228-?00-0602J" device="1277-"/>
-<part name="S1" library="switch" library_urn="urn:adsk.eagle:library:380" deviceset="255SB" device=""/>
 <part name="GND2" library="supply1" library_urn="urn:adsk.eagle:library:371" deviceset="GND" device=""/>
 <part name="CON1" library="pinhead" library_urn="urn:adsk.eagle:library:325" deviceset="PINHD-1X14" device=""/>
@@
 <part name="GND8" library="supply1" library_urn="urn:adsk.eagle:library:371" deviceset="GND" device=""/>
 <part name="GND9" library="supply1" library_urn="urn:adsk.eagle:library:371" deviceset="GND" device=""/>
+<part name="S1" library="switch" deviceset="M251" device=""/>
 </parts>
 <sheets>
@@
 <instance part="MBED" gate="KIT" x="-45.72" y="60.96"/>
 <instance part="ZX2" gate="G$1" x="-27.94" y="-5.08" rot="R90"/>
-<instance part="S1" gate="1" x="17.78" y="86.36" rot="R270"/>
 <instance part="GND2" gate="1" x="-101.6" y="81.28"/>
 <instance part="CON1" gate="A" x="-25.4" y="-22.86" rot="R270"/>
@@
 <instance part="GND8" gate="1" x="25.4" y="-30.48"/>
 <instance part="GND9" gate="1" x="33.02" y="-30.48"/>
+<instance part="S1" gate="1" x="17.78" y="86.36" rot="R270"/>
 </instances>
 <busses>
@@
 <segment>
 <pinref part="MBED" gate="KIT" pin="VO"/>
+<wire x1="2.54" y1="83.82" x2="12.7" y2="83.82" width="0.1524" layer="91"/>
 <pinref part="S1" gate="1" pin="P"/>
-<wire x1="2.54" y1="83.82" x2="12.7" y2="83.82" width="0.1524" layer="91"/>
 </segment>
 </net>
@@
 <net name="BUS0" class="0">
 <segment>
-<pinref part="S1" gate="1" pin="S"/>
 <wire x1="15.24" y1="53.34" x2="22.86" y2="53.34" width="0.1524" layer="91"/>
 <wire x1="22.86" y1="53.34" x2="22.86" y2="81.28" width="0.1524" layer="91"/>
 <pinref part="LED_20P" gate="G$1" pin="A"/>
 <wire x1="22.86" y1="81.28" x2="30.48" y2="81.28" width="0.1524" layer="91"/>
+<pinref part="S1" gate="1" pin="S"/>
 <junction x="22.86" y="81.28"/>
 </segment>
@@
 <net name="BUS8P0" class="0">
 <segment>
-<pinref part="S1" gate="1" pin="O"/>
 <wire x1="22.86" y1="86.36" x2="43.18" y2="86.36" width="0.1524" layer="91"/>
 <wire x1="43.18" y1="86.36" x2="43.18" y2="53.34" width="0.1524" layer="91"/>
@@
 <wire x1="43.18" y1="86.36" x2="53.34" y2="86.36" width="0.1524" layer="91"/>
 <wire x1="53.34" y1="86.36" x2="53.34" y2="81.28" width="0.1524" layer="91"/>
-</segment>
-<segment>
+<pinref part="S1" gate="1" pin="O"/>
+</segment>
+<segment>

Commit message: Update to version2.0
Parts:
- removed JP1, JP2, JP3, JP4, JP5: (no value), jumper:JP2E
- removed R2: (no value), rcl:R-US_0207/10
- added S2: (no value), switch-dil:DIP05YL
Connections:
- removed net N$21: LED_8P.C, R2.2
- net BUS2: now also S2.2; no longer JP2.3
- net BUS3: now also S2.5; no longer JP3.3
- net BUS4: now also S2.4; no longer JP4.3
- net BUS5: now also S2.3; no longer JP5.3
- net BUS8P1: now also S2.10; no longer JP1.2
- net BUS8P2: now also S2.9; no longer JP2.2
- net BUS8P3: now also S2.6; no longer JP3.2
- net BUS8P4: now also S2.7; no longer JP4.2
- net BUS8P5: now also S2.8; no longer JP5.2
- net GND: now also S2.1; no longer JP1.3, R2.1
- net N$2: now also LED_8P.C
Other:
- moved on the sheet: LED_8P
Changed lines of the file:
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@@
 <?xml version="1.0" encoding="utf-8"?>
 <!DOCTYPE eagle SYSTEM "eagle.dtd">
-<eagle version="8.2.2">
+<eagle version="8.7.0">
 <drawing>
 <settings>
-<setting alwaysvectorfont="no"/>
+<setting alwaysvectorfont="yes"/>
+<setting keepoldvectorfont="yes"/>
 <setting verticaltext="up"/>
 </settings>
@@
 <part name="LPC1114" library="lpc1114fn28" deviceset="LPC1114FDH28" device=""/>
 <part name="LED_8P" library="LED" deviceset="LED" device="3MM"/>
-<part name="R2" library="rcl" deviceset="R-US_" device="0207/10"/>
-<part name="GND4" library="supply1" library_urn="urn:adsk.eagle:library:371" deviceset="GND" device=""/>
-<part name="JP2" library="jumper" deviceset="JP2E" device=""/>
-<part name="JP3" library="jumper" deviceset="JP2E" device=""/>
-<part name="JP4" library="jumper" deviceset="JP2E" device=""/>
-<part name="JP5" library="jumper" deviceset="JP2E" device=""/>
-<part name="JP1" library="jumper" deviceset="JP2E" device=""/>
 <part name="GND6" library="supply1" library_urn="urn:adsk.eagle:library:371" deviceset="GND" device=""/>
 <part name="C1" library="rcl" deviceset="C-EU" device="C2012"/>
@@
 <part name="GND9" library="supply1" library_urn="urn:adsk.eagle:library:371" deviceset="GND" device=""/>
 <part name="S1" library="switch" deviceset="M251" device=""/>
+<part name="S2" library="switch-dil" library_urn="urn:adsk.eagle:library:375" deviceset="DIP05YL" device="" package3d_urn="urn:adsk.eagle:package:27259/2"/>
 </parts>
 <sheets>
@@
 <instance part="GND5" gate="1" x="-27.94" y="17.78" rot="R180"/>
 <instance part="LPC1114" gate="G$1" x="-43.18" y="-66.04" rot="R90"/>
-<instance part="LED_8P" gate="G$1" x="53.34" y="78.74"/>
-<instance part="R2" gate="G$1" x="53.34" y="68.58" rot="R90"/>
-<instance part="GND4" gate="1" x="53.34" y="60.96"/>
-<instance part="JP2" gate="1" x="60.96" y="50.8"/>
-<instance part="JP3" gate="1" x="71.12" y="50.8"/>
-<instance part="JP4" gate="1" x="81.28" y="50.8"/>
-<instance part="JP5" gate="1" x="91.44" y="50.8"/>
-<instance part="JP1" gate="1" x="101.6" y="50.8"/>
-<instance part="GND6" gate="1" x="104.14" y="25.4"/>
+<instance part="LED_8P" gate="G$1" x="38.1" y="78.74"/>
+<instance part="GND6" gate="1" x="68.58" y="-5.08"/>
 <instance part="C1" gate="G$1" x="25.4" y="-22.86"/>
 <instance part="C2" gate="G$1" x="33.02" y="-22.86"/>
@@
 <instance part="GND9" gate="1" x="33.02" y="-30.48"/>
 <instance part="S1" gate="1" x="17.78" y="86.36" rot="R270"/>
+<instance part="S2" gate="1" x="73.66" y="25.4"/>
 </instances>
 <busses>
@@
 </segment>
 <segment>
-<pinref part="R2" gate="G$1" pin="1"/>
-<pinref part="GND4" gate="1" pin="GND"/>
-</segment>
-<segment>
-<pinref part="JP1" gate="1" pin="3"/>
-<pinref part="GND6" gate="1" pin="GND"/>
-<wire x1="104.14" y1="27.94" x2="104.14" y2="48.26" width="0.1524" layer="91"/>
-</segment>
-<segment>
 <pinref part="C1" gate="G$1" pin="2"/>
 <pinref part="GND8" gate="1" pin="GND"/>
@@
 <pinref part="C2" gate="G$1" pin="2"/>
 <pinref part="GND9" gate="1" pin="GND"/>
+</segment>
+<segment>
+<pinref part="S2" gate="1" pin="1"/>
+<pinref part="GND6" gate="1" pin="GND"/>
+<wire x1="68.58" y1="17.78" x2="68.58" y2="-2.54" width="0.1524" layer="91"/>
 </segment>
 </net>
@@
 <pinref part="LED_20P" gate="G$1" pin="C"/>
 <pinref part="R1" gate="G$1" pin="2"/>
+<pinref part="LED_8P" gate="G$1" pin="C"/>
+<wire x1="38.1" y1="73.66" x2="30.48" y2="73.66" width="0.1524" layer="91"/>
 </segment>
 </net>
@@
 </segment>
 <segment>
-<pinref part="JP5" gate="1" pin="3"/>
-<wire x1="15.24" y1="17.78" x2="93.98" y2="17.78" width="0.1524" layer="91"/>
-<wire x1="93.98" y1="17.78" x2="93.98" y2="48.26" width="0.1524" layer="91"/>
+<pinref part="S2" gate="1" pin="3"/>
+<wire x1="15.24" y1="12.7" x2="73.66" y2="12.7" width="0.1524" layer="91"/>
+<wire x1="73.66" y1="12.7" x2="73.66" y2="17.78" width="0.1524" layer="91"/>
 </segment>
 </net>
@@
 </segment>
 <segment>
-<pinref part="JP4" gate="1" pin="3"/>
-<wire x1="15.24" y1="20.32" x2="83.82" y2="20.32" width="0.1524" layer="91"/>
-<wire x1="83.82" y1="20.32" x2="83.82" y2="48.26" width="0.1524" layer="91"/>
+<pinref part="S2" gate="1" pin="4"/>
+<wire x1="15.24" y1="10.16" x2="76.2" y2="10.16" width="0.1524" layer="91"/>
+<wire x1="76.2" y1="10.16" x2="76.2" y2="17.78" width="0.1524" layer="91"/>
 </segment>
 </net>
@@
 </segment>
 <segment>
-<pinref part="JP3" gate="1" pin="3"/>
-<wire x1="15.24" y1="22.86" x2="73.66" y2="22.86" width="0.1524" layer="91"/>
-<wire x1="73.66" y1="22.86" x2="73.66" y2="48.26" width="0.1524" layer="91"/>
+<pinref part="S2" gate="1" pin="5"/>
+<wire x1="15.24" y1="7.62" x2="78.74" y2="7.62" width="0.1524" layer="91"/>
+<wire x1="78.74" y1="7.62" x2="78.74" y2="17.78" width="0.1524" layer="91"/>
 </segment>
 </net>
@@
 </segment>
 <segment>
-<pinref part="JP2" gate="1" pin="3"/>
-<wire x1="15.24" y1="25.4" x2="63.5" y2="25.4" width="0.1524" layer="91"/>
-<wire x1="63.5" y1="25.4" x2="63.5" y2="48.26" width="0.1524" layer="91"/>
+<pinref part="S2" gate="1" pin="2"/>
+<wire x1="15.24" y1="15.24" x2="71.12" y2="15.24" width="0.1524" layer="91"/>
+<wire x1="71.12" y1="15.24" x2="71.12" y2="17.78" width="0.1524" layer="91"/>
 </segment>
 </net>
@@
 <net name="BUS8P0" class="0">
 <segment>
-<wire x1="22.86" y1="86.36" x2="43.18" y2="86.36" width="0.1524" layer="91"/>
+<wire x1="22.86" y1="86.36" x2="38.1" y2="86.36" width="0.1524" layer="91"/>
 <wire x1="43.18" y1="86.36" x2="43.18" y2="53.34" width="0.1524" layer="91"/>
 <pinref part="LED_8P" gate="G$1" pin="A"/>
-<wire x1="43.18" y1="86.36" x2="53.34" y2="86.36" width="0.1524" layer="91"/>
-<wire x1="53.34" y1="86.36" x2="53.34" y2="81.28" width="0.1524" layer="91"/>
+<wire x1="43.18" y1="86.36" x2="38.1" y2="86.36" width="0.1524" layer="91"/>
+<wire x1="38.1" y1="86.36" x2="38.1" y2="81.28" width="0.1524" layer="91"/>
 <pinref part="S1" gate="1" pin="O"/>
 </segment>
@@
 </segment>
 </net>
-<net name="N$21" class="0">
-<segment>
-<pinref part="LED_8P" gate="G$1" pin="C"/>
-<pinref part="R2" gate="G$1" pin="2"/>
-</segment>
-</net>
 <net name="BUS8P2" class="0">
 <segment>
@@
 </segment>
 <segment>
-<pinref part="JP2" gate="1" pin="2"/>
-<wire x1="43.18" y1="45.72" x2="60.96" y2="45.72" width="0.1524" layer="91"/>
-<wire x1="60.96" y1="45.72" x2="60.96" y2="48.26" width="0.1524" layer="91"/>
+<pinref part="S2" gate="1" pin="9"/>
+<wire x1="43.18" y1="38.1" x2="71.12" y2="38.1" width="0.1524" layer="91"/>
+<wire x1="71.12" y1="38.1" x2="71.12" y2="33.02" width="0.1524" layer="91"/>
 </segment>
 </net>
@@
 </segment>
 <segment>
-<pinref part="JP3" gate="1" pin="2"/>
-<wire x1="43.18" y1="43.18" x2="71.12" y2="43.18" width="0.1524" layer="91"/>
-<wire x1="71.12" y1="43.18" x2="71.12" y2="48.26" width="0.1524" layer="91"/>
+<pinref part="S2" gate="1" pin="6"/>
+<wire x1="43.18" y1="45.72" x2="78.74" y2="45.72" width="0.1524" layer="91"/>
+<wire x1="78.74" y1="45.72" x2="78.74" y2="33.02" width="0.1524" layer="91"/>
 </segment>
 </net>
@@
 </segment>
 <segment>
-<pinref part="JP4" gate="1" pin="2"/>
-<wire x1="43.18" y1="40.64" x2="81.28" y2="40.64" width="0.1524" layer="91"/>
-<wire x1="81.28" y1="40.64" x2="81.28" y2="48.26" width="0.1524" layer="91"/>
+<pinref part="S2" gate="1" pin="7"/>
+<wire x1="43.18" y1="43.18" x2="76.2" y2="43.18" width="0.1524" layer="91"/>
+<wire x1="76.2" y1="43.18" x2="76.2" y2="33.02" width="0.1524" layer="91"/>
 </segment>
 </net>
@@
 </segment>
 <segment>
-<pinref part="JP5" gate="1" pin="2"/>
-<wire x1="43.18" y1="38.1" x2="91.44" y2="38.1" width="0.1524" layer="91"/>
-<wire x1="91.44" y1="38.1" x2="91.44" y2="48.26" width="0.1524" layer="91"/>
+<pinref part="S2" gate="1" pin="8"/>
+<wire x1="43.18" y1="40.64" x2="73.66" y2="40.64" width="0.1524" layer="91"/>
+<wire x1="73.66" y1="40.64" x2="73.66" y2="33.02" width="0.1524" layer="91"/>
 </segment>
 </net>
@@
 </segment>
 <segment>
-<pinref part="JP1" gate="1" pin="2"/>
-<wire x1="43.18" y1="35.56" x2="101.6" y2="35.56" width="0.1524" layer="91"/>
-<wire x1="101.6" y1="35.56" x2="101.6" y2="48.26" width="0.1524" layer="91"/>
-</segment>
-<segment>
 <wire x1="-53.34" y1="27.94" x2="-53.34" y2="20.32" width="0.1524" layer="91"/>
 <pinref part="C3" gate="G$1" pin="2"/>
 <wire x1="-53.34" y1="20.32" x2="-60.96" y2="20.32" width="0.1524" layer="91"/>
+</segment>
+<segment>
+<wire x1="43.18" y1="35.56" x2="68.58" y2="35.56" width="0.1524" layer="91"/>
+<pinref part="S2" gate="1" pin="10"/>
+<wire x1="68.58" y1="35.56" x2="68.58" y2="33.02" width="0.1524" layer="91"/>
 </segment>
 </net>
@@
 <compatibility>
 <note version="8.2" severity="warning">
-Since Version 8.2, Eagle supports online libraries. The ids
+Since Version 8.2, EAGLE supports online libraries. The ids
 of those online libraries will not be understood (or retained)
 with this version.
 </note>
+<note version="8.3" severity="warning">
+Since Version 8.3, EAGLE supports URNs for individual library
+assets (packages, symbols, and devices). The URNs of those assets
+will not be understood (or retained) with this version.
+</note>
+<note version="8.3" severity="warning">
+Since Version 8.3, EAGLE supports the association of 3D packages
+with devices in libraries, schematics, and board files. Those 3D
+packages will not be understood (or retained) with this version.
+</note>
 </compatibility>
